Commit message: Add Intel RealSense D435 camera to rover.xacro
Added Intel RealSense D435 camera configuration including links, joints, and gazebo sensor settings.

File: ros2_ws/src/rover_bot/urdf/rover.xacro (robot description, xacro)
@@ -181,5 +181,68 @@
     </sensor>
   </gazebo>
-<gazebo reference="base_link">
+  <!-- ───────── Intel RealSense D435 ───────── -->
+  <link name="realsense_link">
+    <visual>
+      <geometry><box size="0.025 0.090 0.025"/></geometry>
+      <material name="dark_grey"><color rgba="0.2 0.2 0.2 1.0"/></material>
+    </visual>
+    <collision>
+      <geometry><box size="0.025 0.090 0.025"/></geometry>
+    </collision>
+    <inertial>
+      <mass value="0.072"/>
+      <inertia ixx="1e-4" ixy="0" ixz="0" iyy="1e-4" iyz="0" izz="1e-4"/>
+    </inertial>
+  </link>
+  <joint name="realsense_joint" type="fixed">
+    <parent link="base_link"/>
+    <child link="realsense_link"/>
+    <origin xyz="0.3 0 0.12" rpy="0 0 0"/>
+  </joint>
+  <!-- Optical frame: Z forward, X right, Y down (ROS convention) -->
+  <link name="realsense_optical_frame"/>
+  <joint name="realsense_optical_joint" type="fixed">
+    <parent link="realsense_link"/>
+    <child link="realsense_optical_frame"/>
+    <origin xyz="0 0 0" rpy="-1.5708 0 -1.5708"/>
+  </joint>
+  <gazebo reference="realsense_link">
+    <sensor name="realsense_d435" type="depth">
+      <always_on>true</always_on>
+      <visualize>true</visualize>
+      <update_rate>30</update_rate>
+      <camera>
+        <horizontal_fov>1.5184</horizontal_fov>
+        <image>
+          <width>640</width>
+          <height>480</height>
+          <format>B8G8R8</format>
+        </image>
+        <clip><near>0.1</near><far>10.0</far></clip>
+        <noise>
+          <type>gaussian</type>
+          <mean>0.0</mean>
+          <stddev>0.005</stddev>
+        </noise>
+      </camera>
+      <plugin name="realsense_plugin" filename="libgazebo_ros_camera.so">
+        <ros>
+          <namespace>/realsense</namespace>
+          <remapping>image_raw:=color/image_raw</remapping>
+          <remapping>camera_info:=color/camera_info</remapping>
+          <remapping>depth/image_raw:=depth/image_rect_raw</remapping>
+          <remapping>depth/camera_info:=depth/camera_info</remapping>
+          <remapping>points:=depth/color/points</remapping>
+        </ros>
+        <camera_name>realsense_d435</camera_name>
+        <frame_name>realsense_optical_frame</frame_name>
+        <hack_baseline>0.07</hack_baseline>
+        <min_depth>0.1</min_depth>
+        <max_depth>10.0</max_depth>
+      </plugin>
+    </sensor>
+  </gazebo>
+  <!-- ──────────────────────────────────────── -->
+  <gazebo reference="base_link">
     <material>Gazebo/Blue</material>
   </gazebo>
